File: PCB-Designs/Modules/8051 board with LCD/8051 with lcd.brd (EAGLE design)
At the start: 6.9 x 7 mm, 30 parts, among them IC1 AT89S51, IC2 7805TV

Commit message: change
Parts:
- moved VR 16.1 mm to (111.8, -2.54), turned to 0 degrees
- moved CONNECTOR 14.0 mm to (115.6, 49.5)
- moved C6 12.7 mm to (94.0, -1.27)
- moved JP1 10.8 mm to (-3.81, 20.3)
- moved S2 10.2 mm to (80.0, -2.54)
- moved CONNECTOR-1 8.89 mm to (68.6, 66.0)
- moved R1 8.89 mm to (76.2, 14.0)
- moved J1 7.62 mm to (-3.81, 44.5)
- moved CONN-6 6.48 mm to (3.81, -3.81)
- moved CONN-7 6.48 mm to (3.81, 5.08)
- moved LED2 4.02 mm to (40.6, -2.54)
- moved CONNECTOR-2 3.81 mm to (40.6, 66.0)
- moved C2 3.81 mm to (88.9, 14.0)
- moved R2 3.81 mm to (25.4, -2.54)
- moved CONNECTOR-4 2.84 mm to (61.0, 21.6)
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Routing:
- net N$39: track 824.1 -> 453.6 mm
- net N$4: track 147.1 -> 224.8 mm
- net N$54: track 62.1 -> 106.7 mm
- net N$3: track 477.5 -> 518.2 mm
- net N$58: track 95.7 -> 134.6 mm
- net N$14: track 81.8 -> 114.8 mm
- net N$48: track 93.5 -> 116.8 mm
- net N$16: track 34.2 -> 56.7 mm
- net N$55: track 65.7 -> 84.1 mm
- net N$5: track 65.9 -> 81.1 mm
- net N$52: track 54.9 -> 69.6 mm
- net N$35: track 88.0 -> 74.0 mm
- net N$51: track 51.3 -> 65.3 mm
- net N$45: track 57.7 -> 45.7 mm
- net N$32: track 47.7 -> 59.5 mm
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