File: PCB-Designs/Modules/4 Channel Relay Board/FOURCHANNEL REAY DRIVER.brd (EAGLE design)
At the start: 103.8 x 85.1 mm, 35 parts, among them T1 BC547, T2 BC547, T3 BC547, T4 BC547

Commit message: change
Parts:
- moved JP6 4.58 mm to (91.4, 67.3)
- moved JP1 3.59 mm to (91.4, 16.5)
- moved JP5 3.59 mm to (91.4, 57.1)
- moved JP4 2.84 mm to (91.4, 47.0)
- moved JP2 2.84 mm to (91.4, 26.7)
- moved JP3 2.54 mm to (91.4, 36.8)
Routing:
- net N$4: track 599.5 -> 626.2 mm
- net N$29: track 254.4 -> 258.7 mm
- net N$13: track 28.4 -> 32.4 mm
- net N$23: track 13.2 -> 16.2 mm
- net N$14: track 13.8 -> 16.3 mm
- net N$26: track 17.0 -> 19.6 mm
- net N$12: track 16.7 -> 18.7 mm
- net N$28: track 20.0 -> 18.7 mm
- net N$11: track 18.3 -> 19.6 mm
- net N$27: track 33.7 -> 34.9 mm
- net N$24: track 28.6 -> 29.8 mm
Other:
- board size 103.8 x 85.1 mm -> 107.6 x 86.4 mm
