File: PCB-Designs/Mini Projects/Hearing Aid/HEARING AID.sch (EAGLE design)
At the start: 22 parts, among them T1 BC547, T2 BC547, T3 BC547, T4 BC547

Commit message: add
Parts:
- removed G1: AB9V, battery:AB9V
- added BATTERY: 9V, battery:AB9V
- added IC1: 7805, v-reg:78XXL
- added R10: 100k, rcl:R-EU_0204/7
- added R8: 10K, rcl:R-EU_0204/7
- added R9: 100E, rcl:R-EU_0204/7
- R3: value (none) -> 1M
- R4: value (none) -> 4.7K
- R5: value (none) -> 3.9K
- R6: value (none) -> 22K; device rcl:R-EU_0204/7 -> resistor:R-TRIMM64P
- R7: value (none) -> 1.5K
- SL1: value (none) -> electret mic
- SL2: value (none) -> ear phone
- SW1: value (none) -> on/off switch
Connections:
- new net N$1: C1.2, R3.2, T1.B
- new net N$10: C5.1, R1.2, R10.2, R4.2, R5.2, R9.1
- new net N$12: C6.1, R6.S
- new net N$13: C6.2, R8.1, T4.B
- new net N$14: R8.2, SL2.2, T4.C
- new net N$16: BATTERY.+, IC1.IN
- new net N$17: BATTERY.-, C4.2, C5.2, D1.A, IC1.GND, R6.E, SL1.1, T1.E, T2.E, T3.E, T4.E
- new net N$18: IC1.OUT, SW1.1
- new net N$19: R9.2, SL2.1, SW1.2
- new net N$2: C1.1, R1.1, SL1.2
- new net N$3: C2.1, R4.1, T1.C
- new net N$4: C2.2, R2.1, T2.B
- new net N$5: C3.1, R2.2, R5.1, T2.C
- new net N$6: C3.2, D1.C, R6.A, T3.B
- new net N$7: R7.1, T3.C
- new net N$8: C4.1, R10.1, R3.1, R7.2
Other:
- moved on the sheet: C1, C2, C3, C4, C5, C6, D1, R1, R2, R3, R4, R5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

Commit message: change
Parts:
- removed SL2: ear phone, con-amp-quick:M02
- added J1: DCJ0202, con-jack:DCJ0202
Connections:
- net N$14: now also J1.3; no longer SL2.2
- net N$19: now also J1.1; no longer SL2.1
Changed lines of the file:
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@@
 <part name="BATTERY" library="battery" deviceset="AB9V" device="" value="9V"/>
 <part name="SL1" library="con-amp-quick" deviceset="M02" device="" value="electret mic"/>
-<part name="SL2" library="con-amp-quick" deviceset="M02" device="" value="ear phone"/>
 <part name="C5" library="capacitor-wima" deviceset="C" device="2.5/6" value="100uf"/>
 <part name="C6" library="capacitor-wima" deviceset="C" device="2.5/6" value="1uf"/>
@@
 <part name="R10" library="rcl" deviceset="R-EU_" device="0204/7" value="100k"/>
 <part name="IC1" library="v-reg" deviceset="78XXL" device="" value="7805"/>
+<part name="J1" library="con-jack" deviceset="DCJ0202" device=""/>
 </parts>
 <sheets>
@@
 <instance part="BATTERY" gate="G$1" x="205.74" y="58.42" rot="R90"/>
 <instance part="SL1" gate="G$1" x="22.86" y="48.26"/>
-<instance part="SL2" gate="G$1" x="149.86" y="66.04" rot="R180"/>
 <instance part="C5" gate="G$1" x="109.22" y="66.04"/>
 <instance part="C6" gate="G$1" x="124.46" y="45.72" rot="R90"/>
@@
 <instance part="R10" gate="G$1" x="96.52" y="71.12" rot="R90"/>
 <instance part="IC1" gate="A" x="185.42" y="71.12" rot="R180"/>
+<instance part="J1" gate="G$1" x="134.62" y="66.04"/>
 </instances>
 <busses>
@@
 <wire x1="101.6" y1="33.02" x2="101.6" y2="55.88" width="0.1524" layer="91"/>
 <wire x1="101.6" y1="55.88" x2="96.52" y2="55.88" width="0.1524" layer="91"/>
+<junction x="96.52" y="55.88"/>
 </segment>
 </net>
@@
 <wire x1="132.08" y1="55.88" x2="139.7" y2="55.88" width="0.1524" layer="91"/>
 <wire x1="139.7" y1="55.88" x2="139.7" y2="50.8" width="0.1524" layer="91"/>
-<pinref part="SL2" gate="G$1" pin="2"/>
 <wire x1="139.7" y1="50.8" x2="139.7" y2="48.26" width="0.1524" layer="91"/>
 <wire x1="139.7" y1="55.88" x2="142.24" y2="55.88" width="0.1524" layer="91"/>
-<wire x1="142.24" y1="55.88" x2="142.24" y2="63.5" width="0.1524" layer="91"/>
 <pinref part="T4" gate="G$1" pin="C"/>
 <junction x="139.7" y="50.8"/>
+<pinref part="J1" gate="G$1" pin="3"/>
+<wire x1="142.24" y1="63.5" x2="142.24" y2="55.88" width="0.1524" layer="91"/>
 </segment>
 </net>
@@
 <wire x1="172.72" y1="73.66" x2="175.26" y2="73.66" width="0.1524" layer="91"/>
 <wire x1="175.26" y1="73.66" x2="175.26" y2="81.28" width="0.1524" layer="91"/>
-<pinref part="SL2" gate="G$1" pin="1"/>
-<wire x1="142.24" y1="66.04" x2="142.24" y2="73.66" width="0.1524" layer="91"/>
 <pinref part="R9" gate="G$1" pin="2"/>
 <wire x1="142.24" y1="73.66" x2="142.24" y2="76.2" width="0.1524" layer="91"/>
@@
 <wire x1="175.26" y1="81.28" x2="142.24" y2="81.28" width="0.1524" layer="91"/>
 <wire x1="142.24" y1="81.28" x2="142.24" y2="73.66" width="0.1524" layer="91"/>
-</segment>
-</net>
+<pinref part="J1" gate="G$1" pin="1"/>
+<wire x1="142.24" y1="73.66" x2="142.24" y2="68.58" width="0.1524" layer="91"/>
+</segment>
+</net>
