File: PCB-Designs/Modules/Arduino with relay driver/arduino.sch (EAGLE design)
At the start: 40 parts, among them T1 BC547, T2 BC547, T3 BC547, T4 BC547

Commit message: made by shankar
Parts:
- removed JP4, JP8: (no value), jumper:JP2E
- added C1, C2: 22pf, capacitor-wima:C2.5/2
- added C3: 100UF, capacitor-wima:C2.5/2
- added C4, C5: 0.1uf, capacitor-wima:C2.5/2
- added C6: 4.7uf, capacitor-wima:C2.5/2
- added D4: 1N4007, diode:1N4004
- added IC1: ATMEGA328, quantum-research-group:QT9701BD
- added IC2: 7805, linear:786TV
- added J1: (no value), con-jack:DCJ0303
- added JP10, JP9: (no value), jumper:JP2E
- added JP13, JP14: (no value), jumper:JP4E
- added LED1, LED2: (no value), led:LED3MM
- added Q1: 12MHZ, crystal:CRYSTALHC49S
- added R1: 220R, rcl:R-EU_0207/10
- added R2: 330R, rcl:R-EU_0207/10
- added R4: 10K, rcl:R-EU_0207/10
- added S1: (no value), switch-dil:DP02
Connections:
- removed net N$16: GR2.1, JP4.1, RG2.2
- removed net N$2: D1.C, D2.C, D3.C, D5.C, JP4.3, RELAY11.2, RELAY21.2, RELAY31.2, RELAY41.2, RR1.2, RR2.2, RR3.2, RR4.2
- removed net N$23: GREEN1.C, GREEN2.C, GREEN3.C, GREEN4.C, JP8.1, RED1.C, RED2.C, RED3.C, RED4.C, T1.E, T2.E, T3.E, T4.E
- removed net N$25: GR3.1, JP8.3, RG3.2
- removed net N$34: GR4.1, JP8.2, RG4.2
- removed net N$6: GR1.1, JP4.2, RG1.2
- new net N$14: C2.2, IC1.XT2, Q1.1
- new net N$21: C1.1, C2.1, C3.2, C4.2, C5.2, C6.2, GREEN1.C, GREEN2.C, GREEN3.C, GREEN4.C, IC1.VSS, IC1.XFR, IC2.GND, J1.2, J1.3, LED1.C, LED2.C, RED1.C, RED2.C, RED3.C, RED4.C, S1.4, T1.E, T2.E, T3.E, T4.E
- new net N$32: C3.1, C4.1, D4.C, IC2.VI
- new net N$39: D4.A, J1.1
- new net N$4: C1.2, IC1.XT1, Q1.2
- new net N$40: C5.1, C6.1, D1.C, D2.C, D3.C, D5.C, IC1.ECS, IC1.VDD@1, IC2.VO, R1.2, R4.2, RELAY11.2, RELAY21.2, RELAY31.2, RELAY41.2, RR1.2, RR2.2, RR3.2, RR4.2
- new net N$41: LED1.A, R1.1
- new net N$42: IC1.SMP, JP9.1
- new net N$43: IC1.Z4, JP9.2
- new net N$44: IC1.Z3, JP9.3
- new net N$45: IC1.Z2, JP10.1
- new net N$46: IC1.Z1, JP10.2
- new net N$47: IC1.CSR, JP10.3
- new net N$48: IC1.AIN, JP14.4
- new net N$49: IC1.OUT, JP14.3
- new net N$50: IC1.STAT, JP14.2
- new net N$51: IC1.BG, JP14.1
- new net N$52: IC1.OBJ, JP13.4
- new net N$53: IC1.DA1/EDI, JP13.2
- new net N$54: IC1.DA0/ECK, JP13.3
- new net N$55: IC1.DA2/EDO, JP13.1, R2.2
- new net N$56: GR4.1, IC1.DA3, RG4.2
- new net N$57: GR3.1, IC1.DA4, RG3.2
- new net N$58: GR2.1, IC1.DA5, RG2.2
- new net N$59: GR1.1, IC1.DA6, RG1.2
- new net N$60: IC1.DA7
- new net N$61: IC1.VSS@1
- new net N$62: IC1.VDD, R4.1, S1.2
- new net N$63: LED2.A, R2.1
Other:
- moved on the sheet: D1, D2, D3, D5, GR1, GR2, GR3, GR4, GREEN1, GREEN2, GREEN3, GREEN4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

Commit message: updated with finising
Parts:
- removed JP13: (no value), jumper:JP4E
- added JP4: (no value), jumper:JP4E
Connections:
- removed net N$48: IC1.AIN, JP14.4
- removed net N$49: IC1.OUT, JP14.3
- removed net N$51: IC1.BG, JP14.1
- removed net N$52: IC1.OBJ, JP13.4
- removed net N$53: IC1.DA1/EDI, JP13.2
- removed net N$54: IC1.DA0/ECK, JP13.3
- new net N$2: JP1.1
- net N$21: now also JP14.1
- net N$26: no longer JP1.1
- net N$30: no longer RELAY41.1
- net N$55: no longer JP13.1
Changed lines of the file:
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@@
 <part name="JP9" library="jumper" deviceset="JP2E" device=""/>
 <part name="JP10" library="jumper" deviceset="JP2E" device=""/>
-<part name="JP13" library="jumper" deviceset="JP4E" device=""/>
 <part name="JP14" library="jumper" deviceset="JP4E" device=""/>
 <part name="R4" library="rcl" deviceset="R-EU_" device="0207/10" value="10K"/>
+<part name="JP4" library="jumper" deviceset="JP4E" device=""/>
 </parts>
 <sheets>
@@
 <instance part="JP9" gate="1" x="76.2" y="104.14" rot="R270"/>
 <instance part="JP10" gate="1" x="76.2" y="96.52" rot="R270"/>
-<instance part="JP13" gate="G$1" x="20.32" y="88.9" rot="R90"/>
 <instance part="JP14" gate="G$1" x="20.32" y="99.06" rot="R90"/>
 <instance part="R4" gate="G$1" x="35.56" y="111.76" rot="R90"/>
+<instance part="JP4" gate="G$1" x="17.78" y="58.42" rot="R90"/>
 </instances>
 <busses>
@@
 <wire x1="180.34" y1="58.42" x2="226.06" y2="58.42" width="0.1524" layer="91"/>
 <junction x="180.34" y="58.42"/>
-<wire x1="226.06" y1="58.42" x2="226.06" y2="73.66" width="0.1524" layer="91"/>
-<pinref part="JP1" gate="A" pin="1"/>
-<wire x1="226.06" y1="73.66" x2="233.68" y2="73.66" width="0.1524" layer="91"/>
-<junction x="233.68" y="73.66"/>
 </segment>
 </net>
@@
 <wire x1="152.4" y1="7.62" x2="165.1" y2="7.62" width="0.1524" layer="91"/>
 <wire x1="165.1" y1="7.62" x2="165.1" y2="20.32" width="0.1524" layer="91"/>
-<pinref part="RELAY4" gate="1" pin="1"/>
-<wire x1="165.1" y1="20.32" x2="177.8" y2="20.32" width="0.1524" layer="91"/>
-<junction x="177.8" y="20.32"/>
 <junction x="152.4" y="7.62"/>
 </segment>
@@
 <junction x="-2.54" y="66.04"/>
 <junction x="-5.08" y="66.04"/>
+<wire x1="10.16" y1="83.82" x2="10.16" y2="91.44" width="0.1524" layer="91"/>
+<pinref part="JP14" gate="G$1" pin="1"/>
+<wire x1="10.16" y1="91.44" x2="22.86" y2="91.44" width="0.1524" layer="91"/>
+<wire x1="22.86" y1="91.44" x2="22.86" y2="96.52" width="0.1524" layer="91"/>
+<junction x="22.86" y="96.52"/>
 </segment>
 </net>
@@
 <wire x1="55.88" y1="86.36" x2="55.88" y2="91.44" width="0.1524" layer="91"/>
 <junction x="71.12" y="86.36"/>
-<junction x="43.18" y="91.44"/>
 <junction x="55.88" y="91.44"/>
 <pinref part="R4" gate="G$1" pin="2"/>
@@
 <junction x="241.3" y="132.08"/>
 <junction x="55.88" y="137.16"/>
+<junction x="43.18" y="91.44"/>
 </segment>
 </net>
@@
 </segment>
 </net>
-<net name="N$48" class="0">
-<segment>
-<pinref part="IC1" gate="G$1" pin="AIN"/>
-<pinref part="JP14" gate="G$1" pin="4"/>
-<wire x1="43.18" y1="104.14" x2="22.86" y2="104.14" width="0.1524" layer="91"/>
-<junction x="43.18" y="104.14"/>
-<junction x="22.86" y="104.14"/>
-</segment>
-</net>
-<net name="N$49" class="0">
-<segment>
-<pinref part="IC1" gate="G$1" pin="OUT"/>
-<pinref part="JP14" gate="G$1" pin="3"/>
-<wire x1="43.18" y1="101.6" x2="22.86" y2="101.6" width="0.1524" layer="91"/>
-<junction x="43.18" y="101.6"/>
-<junction x="22.86" y="101.6"/>
-</segment>
-</net>
-<net name="N$50" class="0">
-<segment>
-<pinref part="IC1" gate="G$1" pin="STAT"/>
-<pinref part="JP14" gate="G$1" pin="2"/>
-<wire x1="43.18" y1="99.06" x2="22.86" y2="99.06" width="0.1524" layer="91"/>
-<junction x="43.18" y="99.06"/>
-<junction x="22.86" y="99.06"/>
-</segment>
-</net>
-<net name="N$51" class="0">
-<segment>
-<pinref part="JP14" gate="G$1" pin="1"/>
-<wire x1="22.86" y1="96.52" x2="43.18" y2="96.52" width="0.1524" layer="91"/>
-<pinref part="IC1" gate="G$1" pin="BG"/>
-<junction x="43.18" y="96.52"/>
-<junction x="22.86" y="96.52"/>
-</segment>
-</net>
-<net name="N$52" class="0">
-<segment>
-<pinref part="JP13" gate="G$1" pin="4"/>
-<pinref part="IC1" gate="G$1" pin="OBJ"/>
-<wire x1="22.86" y1="93.98" x2="43.18" y2="93.98" width="0.1524" layer="91"/>
-<junction x="43.18" y="93.98"/>
-<junction x="22.86" y="93.98"/>
-</segment>
-</net>
-<net name="N$53" class="0">
-<segment>
-<pinref part="IC1" gate="G$1" pin="DA1/EDI"/>
-<pinref part="JP13" gate="G$1" pin="2"/>
-<wire x1="38.1" y1="78.74" x2="43.18" y2="78.74" width="0.1524" layer="91"/>
-<wire x1="22.86" y1="88.9" x2="38.1" y2="88.9" width="0.1524" layer="91"/>
-<wire x1="38.1" y1="88.9" x2="38.1" y2="78.74" width="0.1524" layer="91"/>
-<junction x="43.18" y="78.74"/>
-<junction x="22.86" y="88.9"/>
-</segment>
-</net>
-<net name="N$54" class="0">
-<segment>
-<pinref part="JP13" gate="G$1" pin="3"/>
-<wire x1="22.86" y1="91.44" x2="40.64" y2="91.44" width="0.1524" layer="91"/>
-<wire x1="40.64" y1="91.44" x2="40.64" y2="81.28" width="0.1524" layer="91"/>
-<pinref part="IC1" gate="G$1" pin="DA0/ECK"/>
-<wire x1="40.64" y1="81.28" x2="43.18" y2="81.28" width="0.1524" layer="91"/>
-<junction x="43.18" y="81.28"/>
-<junction x="22.86" y="91.44"/>
-</segment>
-</net>
 <net name="N$55" class="0">
 <segment>
-<pinref part="JP13" gate="G$1" pin="1"/>
-<wire x1="22.86" y1="86.36" x2="22.86" y2="76.2" width="0.1524" layer="91"/>
 <pinref part="IC1" gate="G$1" pin="DA2/EDO"/>
-<wire x1="22.86" y1="76.2" x2="30.48" y2="76.2" width="0.1524" layer="91"/>
 <junction x="43.18" y="76.2"/>
-<junction x="22.86" y="86.36"/>
 <pinref part="R2" gate="G$1" pin="2"/>
 <wire x1="30.48" y1="76.2" x2="43.18" y2="76.2" width="0.1524" layer="91"/>
@@
 </segment>
 </net>
+<net name="N$2" class="0">
+<segment>
+<pinref part="JP1" gate="A" pin="1"/>
+<junction x="233.68" y="73.66"/>
+<wire x1="226.06" y1="73.66" x2="233.68" y2="73.66" width="0.1524" layer="91"/>
+</segment>
+</net>
+<net name="N$23" class="0">
+<segment>
+<pinref part="IC1" gate="G$1" pin="STAT"/>
+<pinref part="JP14" gate="G$1" pin="2"/>
+<wire x1="43.18" y1="99.06" x2="22.86" y2="99.06" width="0.1524" layer="91"/>
+<junction x="22.86" y="99.06"/>
+<junction x="43.18" y="99.06"/>
+</segment>
+</net>
