File: PCB-Designs/Modules/Arduino with relay driver/arduino.brd (EAGLE design)
At the start: 144.8 x 150.8 mm, 40 parts, among them T1 BC547, T2 BC547, T3 BC547, T4 BC547

Commit message: made by shankar
Parts:
- removed JP4, JP8: (no value), jumper:JP2
- added C1, C2: 22pf, capacitor-wima:C2.5-2
- added C3: 100UF, capacitor-wima:C2.5-2
- added C4, C5: 0.1uf, capacitor-wima:C2.5-2
- added C6: 4.7uf, capacitor-wima:C2.5-2
- added D4: 1N4007, diode:DO41-10
- added IC1: ATMEGA328, quantum-research-group:DIL28-3
- added IC2: 7805, linear:TO220V
- added J1: (no value), con-jack:DCJ0303
- added JP10, JP9: (no value), jumper:JP2
- added JP13, JP14: (no value), jumper:JP4
- added LED1, LED2: (no value), led:LED3MM
- added Q1: 12MHZ, crystal:HC49/S
- added R1: 220R, rcl:0207/10
- added R2: 330R, rcl:0207/10
- added R4: 10K, rcl:0207/10
- added S1: (no value), switch-dil:DP-02
- moved D3 170.4 mm to (215.9, -35.6)
- moved D1 168.9 mm to (215.9, 69.8)
- moved D2 168.9 mm to (215.9, 5.08)
- moved D5 168.9 mm to (215.9, 38.1)
- moved GR1 168.9 mm to (246.4, 71.1)
- moved GR2 168.9 mm to (246.4, 39.4)
- moved GR3 168.9 mm to (246.4, 5.08)
- moved GR4 168.9 mm to (246.4, -30.5)
- moved GREEN1 168.9 mm to (260.4, 57.1)
- moved GREEN2 168.9 mm to (261.6, 25.4)
- moved GREEN3 168.9 mm to (261.6, -7.62)
- moved GREEN4 168.9 mm to (261.6, -41.9)
- moved RED1 168.9 mm to (278.1, 85.1)
- moved RED2 168.9 mm to (278.1, 50.8)
- moved RED3 168.9 mm to (278.1, 16.5)
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Connections:
- removed net N$16: GR2.1, JP4.1, RG2.2
- removed net N$2: D1.C, D2.C, D3.C, D5.C, JP4.3, RELAY1.2, RELAY2.2, RELAY3.2, RELAY4.2, RR1.2, RR2.2, RR3.2, RR4.2
- removed net N$23: GREEN1.K, GREEN2.K, GREEN3.K, GREEN4.K, JP8.1, RED1.K, RED2.K, RED3.K, RED4.K, T1.1, T2.1, T3.1, T4.1
- removed net N$25: GR3.1, JP8.3, RG3.2
- removed net N$34: GR4.1, JP8.2, RG4.2
- removed net N$6: GR1.1, JP4.2, RG1.2
- new net N$14: C2.2, IC1.10, Q1.1
- new net N$21: C1.1, C2.1, C3.2, C4.2, C5.2, C6.2, GREEN1.K, GREEN2.K, GREEN3.K, GREEN4.K, IC1.22, IC1.8, IC2.2, J1.2, J1.3, LED1.K, LED2.K, RED1.K, RED2.K, RED3.K, RED4.K, S1.4, T1.1, T2.1, T3.1, T4.1
- new net N$32: C3.1, C4.1, D4.C, IC2.1
- new net N$39: D4.A, J1.1
- new net N$4: C1.2, IC1.9, Q1.2
- new net N$40: C5.1, C6.1, D1.C, D2.C, D3.C, D5.C, IC1.20, IC1.7, IC2.3, R1.2, R4.2, RELAY1.2, RELAY2.2, RELAY3.2, RELAY4.2, RR1.2, RR2.2, RR3.2, RR4.2
- new net N$41: LED1.A, R1.1
- new net N$42: IC1.28, JP9.1
- new net N$43: IC1.27, JP9.2
- new net N$44: IC1.26, JP9.3
- new net N$45: IC1.25, JP10.1
- new net N$46: IC1.24, JP10.2
- new net N$47: IC1.23, JP10.3
- new net N$48: IC1.2, JP14.4
- new net N$49: IC1.3, JP14.3
- new net N$50: IC1.4, JP14.2
- new net N$51: IC1.5, JP14.1
- new net N$52: IC1.6, JP13.4
- new net N$53: IC1.12, JP13.2
- new net N$54: IC1.11, JP13.3
- new net N$55: IC1.13, JP13.1, R2.2
- new net N$56: GR4.1, IC1.14, RG4.2
- new net N$57: GR3.1, IC1.15, RG3.2
- new net N$58: GR2.1, IC1.16, RG2.2
- new net N$59: GR1.1, IC1.17, RG1.2
- new net N$60: IC1.18
- new net N$61: IC1.19
- new net N$62: IC1.1, R4.1, S1.2
- new net N$63: LED2.A, R2.1
Routing:
- net N$21: track 0.00 -> 1560.7 mm
- net N$40: track 0.00 -> 1117.6 mm
- net N$57: track 0.00 -> 931.4 mm
- net N$56: track 0.00 -> 806.0 mm
- net N$23: track 719.5 -> 0.00 mm
- net N$2: track 586.7 -> 0.00 mm
- net N$59: track 0.00 -> 407.5 mm
- net N$58: track 0.00 -> 401.1 mm
- net N$16: track 342.9 -> 0.00 mm
- net N$34: track 341.0 -> 0.00 mm
- net N$6: track 307.9 -> 0.00 mm
- net N$55: track 0.00 -> 158.7 mm
- net N$62: track 0.00 -> 135.9 mm
- net N$25: track 100.5 -> 0.00 mm
- net N$14: track 0.00 -> 54.0 mm
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Other:
- board size 144.8 x 150.8 mm -> 7.1 x 7 mm

Commit message: updated with finising
Parts:
- removed JP13: (no value), jumper:JP4
- added JP4: (no value), jumper:JP4
- moved C5 5.08 mm to (120.7, 77.5)
- moved C6 5.08 mm to (132.1, 77.5)
- moved GREEN2 3.81 mm to (261.6, 21.6)
- moved RG2 3.81 mm to (274.3, 21.6)
- moved RED3 2.84 mm to (279.4, 14.0)
- moved C2 2.54 mm to (95.2, 25.4)
- moved GREEN1 2.54 mm to (260.4, 54.6)
- moved RG1 1.27 mm to (274.3, 54.6)
- moved RG4 1.27 mm to (275.6, -44.5)
- moved RED2 1.27 mm to (278.1, 49.5)
- moved RR2 1.27 mm to (265.4, 49.5)
Connections:
- removed net N$48: IC1.2, JP14.4
- removed net N$49: IC1.3, JP14.3
- removed net N$51: IC1.5, JP14.1
- removed net N$52: IC1.6, JP13.4
- removed net N$53: IC1.12, JP13.2
- removed net N$54: IC1.11, JP13.3
- new net N$2: JP1.1
- net N$21: now also JP14.1
- net N$26: no longer JP1.1
- net N$30: no longer RELAY4.1
- net N$55: no longer JP13.1
Routing:
- net N$21: track 1560.7 -> 1644.7 mm
- net N$56: track 806.0 -> 857.3 mm
- net N$55: track 158.7 -> 110.5 mm
- net N$54: track 46.0 -> 0.00 mm
- net N$57: track 931.4 -> 976.1 mm
- net N$53: track 30.8 -> 0.00 mm
- net N$26: track 56.1 -> 30.7 mm, vias 0 -> 1
- net N$52: track 22.9 -> 0.00 mm
- net N$58: track 401.1 -> 424.0 mm
- net N$30: track 79.1 -> 58.4 mm, vias 0 -> 1
- net N$62: track 135.9 -> 156.2 mm
- net N$51: track 20.3 -> 0.00 mm
- net N$49: track 20.3 -> 0.00 mm
- net N$48: track 20.3 -> 0.00 mm
- net N$16: track 0.00 -> 14.0 mm, vias 0 -> 1
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
Commit message: updated
Parts:
- moved JP4 2.54 mm to (113.0, 24.1)
Routing:
- net N$12: track 58.7 -> 60.2 mm
Changed lines of the file:
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@@
 <element name="JP14" library="jumper" package="JP4" value="" x="113.03" y="57.15" rot="R90"/>
 <element name="R4" library="rcl" package="0207/10" value="10K" x="142.24" y="86.36" rot="R270"/>
-<element name="JP4" library="jumper" package="JP4" value="" x="113.03" y="21.59" rot="R90"/>
+<element name="JP4" library="jumper" package="JP4" value="" x="113.03" y="24.13" rot="R90"/>
 </elements>
 <signals>
@@
 <wire x1="259.08" y1="1.27" x2="259.08" y2="-1.27" width="1.016" layer="16"/>
 <wire x1="259.08" y1="-1.27" x2="261.62" y2="-1.27" width="1.016" layer="16"/>
-<wire x1="232.41" y1="8.89" x2="232.41" y2="11.43" width="1.016" layer="16"/>
-<wire x1="232.41" y1="11.43" x2="248.92" y2="11.43" width="1.016" layer="16"/>
+<wire x1="232.41" y1="8.89" x2="231.14" y2="11.43" width="1.016" layer="16"/>
+<wire x1="231.14" y1="11.43" x2="248.92" y2="11.43" width="1.016" layer="16"/>
 <wire x1="261.62" y1="-1.27" x2="261.747" y2="-2.159" width="0.254" layer="16"/>
 </signal>
@@
 <wire x1="60.96" y1="63.5" x2="63.5" y2="63.5" width="1.016" layer="16"/>
 <wire x1="60.96" y1="-25.4" x2="60.96" y2="63.5" width="1.016" layer="16"/>
-<wire x1="170.18" y1="-25.4" x2="60.96" y2="-25.4" width="1.016" layer="16"/>
-<wire x1="198.12" y1="24.13" x2="170.18" y2="24.13" width="1.016" layer="16"/>
-<wire x1="170.18" y1="24.13" x2="170.18" y2="-25.4" width="1.016" layer="16"/>
+<wire x1="176.53" y1="-25.4" x2="60.96" y2="-25.4" width="1.016" layer="16"/>
+<wire x1="198.12" y1="24.13" x2="176.53" y2="24.13" width="1.016" layer="16"/>
+<wire x1="176.53" y1="24.13" x2="176.53" y2="-25.4" width="1.016" layer="16"/>
 <wire x1="198.12" y1="90.17" x2="198.12" y2="24.13" width="1.016" layer="16"/>
 <wire x1="312.42" y1="90.17" x2="198.12" y2="90.17" width="1.016" layer="16"/>
