File: pcb_designs/modules/dtmf_module/DTMF.brd (EAGLE design)
At the start: 50.5 x 55.9 mm, 18 parts, among them IC1 CM8870CP

Commit message: 
Parts:
- C1: value 0.47uf -> 0.1uf
Changed lines of the file:
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@@
 <?xml version="1.0" encoding="utf-8"?>
 <!DOCTYPE eagle SYSTEM "eagle.dtd">
-<eagle version="6.5.0">
+<eagle version="6.1">
 <drawing>
 <settings>
@@
 <layer number="21" name="tPlace" color="7" fill="1" visible="yes" active="yes"/>
 <layer number="22" name="bPlace" color="7" fill="1" visible="yes" active="yes"/>
-<layer number="23" name="tOrigins" color="15" fill="1" visible="no" active="yes"/>
+<layer number="23" name="tOrigins" color="15" fill="1" visible="yes" active="yes"/>
 <layer number="24" name="bOrigins" color="15" fill="1" visible="yes" active="yes"/>
 <layer number="25" name="tNames" color="7" fill="1" visible="yes" active="yes"/>
@@
 </class>
 </classes>
-<designrules name="default *">
+<designrules>
 <description language="de">&lt;b&gt;EAGLE Design Rules&lt;/b&gt;
 &lt;p&gt;
@@
 <element name="R1" library="rcl" package="0204/7" value="10K" x="25.4" y="53.34" rot="R180"/>
 <element name="R2" library="rcl" package="0204/7" value="100K" x="34.29" y="48.26"/>
-<element name="C1" library="capacitor-wima" package="C2.5-2" value="0.47uf" x="35.56" y="54.61" rot="R270"/>
+<element name="C1" library="capacitor-wima" package="C2.5-2" value="0.1uf" x="35.56" y="54.61" rot="R270"/>
 <element name="C2" library="capacitor-wima" package="C2.5-2" value="22PF" x="26.67" y="38.1" rot="R180"/>
 <element name="C3" library="capacitor-wima" package="C2.5-2" value="22PF" x="26.67" y="31.75" rot="R180"/>
