File: pcb_designs/pic/pic_board/pic_board.sch (EAGLE design)
At the start: 22 parts, among them IC1 PIC16f877a, IC2 7805TV

Commit message: modify
Parts:
- added R3: 10K, rcl:R-EU_0204/7
- added SL1, SL2: 4 pin, con-amp-quick:M04
Connections:
- new net N$39: IC1.!MCLR!/VPP/RE3, R3.2
- net N$33: now also R3.1, SL2.1, SL2.2, SL2.3, SL2.4; no longer IC1.!MCLR!/VPP/RE3
- net N$35: now also SL1.1, SL1.2, SL1.3, SL1.4
Changed lines of the file:
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@@
 <attribute name="OC_NEWARK" value="unknown"/>
 </part>
+<part name="SL1" library="con-amp-quick" deviceset="M04" device="" value="4 pin"/>
+<part name="SL2" library="con-amp-quick" deviceset="M04" device="" value="4 pin"/>
+<part name="R3" library="rcl" deviceset="R-EU_" device="0204/7" value="10K"/>
 </parts>
 <sheets>
@@
 <instance part="LED2" gate="G$1" x="10.16" y="73.66" rot="R180"/>
 <instance part="CONNECTOR1" gate="G$1" x="132.08" y="43.18" rot="R180"/>
+<instance part="SL1" gate="G$1" x="-7.62" y="45.72"/>
+<instance part="SL2" gate="G$1" x="12.7" y="86.36"/>
+<instance part="R3" gate="G$1" x="22.86" y="93.98"/>
 </instances>
 <busses>
@@
 <pinref part="IC1" gate="G$1" pin="VDD@1"/>
 <wire x1="93.98" y1="63.5" x2="116.84" y2="63.5" width="0.1524" layer="91"/>
-<pinref part="IC1" gate="G$1" pin="!MCLR!/VPP/RE3"/>
-<wire x1="45.72" y1="83.82" x2="45.72" y2="93.98" width="0.1524" layer="91"/>
-<wire x1="45.72" y1="93.98" x2="17.78" y2="93.98" width="0.1524" layer="91"/>
-<wire x1="17.78" y1="93.98" x2="17.78" y2="60.96" width="0.1524" layer="91"/>
+<wire x1="17.78" y1="93.98" x2="17.78" y2="91.44" width="0.1524" layer="91"/>
 <pinref part="R2" gate="G$1" pin="2"/>
 <junction x="10.16" y="60.96"/>
 <pinref part="IC1" gate="G$1" pin="VDD"/>
+<wire x1="17.78" y1="91.44" x2="17.78" y2="88.9" width="0.1524" layer="91"/>
+<wire x1="17.78" y1="88.9" x2="17.78" y2="86.36" width="0.1524" layer="91"/>
+<wire x1="17.78" y1="86.36" x2="17.78" y2="83.82" width="0.1524" layer="91"/>
+<wire x1="17.78" y1="83.82" x2="17.78" y2="60.96" width="0.1524" layer="91"/>
 <wire x1="45.72" y1="58.42" x2="66.04" y2="58.42" width="0.1524" layer="91"/>
 <wire x1="66.04" y1="58.42" x2="66.04" y2="60.96" width="0.1524" layer="91"/>
 <wire x1="66.04" y1="60.96" x2="86.36" y2="60.96" width="0.1524" layer="91"/>
+<pinref part="SL2" gate="G$1" pin="1"/>
+<junction x="17.78" y="83.82"/>
+<pinref part="SL2" gate="G$1" pin="2"/>
+<junction x="17.78" y="86.36"/>
+<pinref part="SL2" gate="G$1" pin="3"/>
+<junction x="17.78" y="88.9"/>
+<pinref part="SL2" gate="G$1" pin="4"/>
+<junction x="17.78" y="91.44"/>
+<pinref part="R3" gate="G$1" pin="1"/>
 </segment>
 </net>
@@
 <junction x="-25.4" y="48.26"/>
 <wire x1="-17.78" y1="38.1" x2="-2.54" y2="38.1" width="0.1524" layer="91"/>
-<wire x1="-2.54" y1="38.1" x2="-2.54" y2="53.34" width="0.1524" layer="91"/>
+<wire x1="-2.54" y1="38.1" x2="-2.54" y2="43.18" width="0.1524" layer="91"/>
 <pinref part="IC2" gate="A1" pin="GND"/>
+<wire x1="-2.54" y1="43.18" x2="-2.54" y2="45.72" width="0.1524" layer="91"/>
+<wire x1="-2.54" y1="45.72" x2="-2.54" y2="48.26" width="0.1524" layer="91"/>
+<wire x1="-2.54" y1="48.26" x2="-2.54" y2="50.8" width="0.1524" layer="91"/>
+<wire x1="-2.54" y1="50.8" x2="-2.54" y2="53.34" width="0.1524" layer="91"/>
 <wire x1="10.16" y1="38.1" x2="-2.54" y2="38.1" width="0.1524" layer="91"/>
 <pinref part="C1" gate="G$1" pin="1"/>
@@
 <pinref part="IC1" gate="G$1" pin="VSS"/>
 <wire x1="45.72" y1="55.88" x2="81.28" y2="55.88" width="0.1524" layer="91"/>
+<pinref part="SL1" gate="G$1" pin="1"/>
+<junction x="-2.54" y="43.18"/>
+<pinref part="SL1" gate="G$1" pin="2"/>
+<junction x="-2.54" y="45.72"/>
+<pinref part="SL1" gate="G$1" pin="3"/>
+<junction x="-2.54" y="48.26"/>
+<pinref part="SL1" gate="G$1" pin="4"/>
+<junction x="-2.54" y="50.8"/>
 </segment>
 </net>
@@
 </segment>
 </net>
+<net name="N$39" class="0">
+<segment>
+<pinref part="IC1" gate="G$1" pin="!MCLR!/VPP/RE3"/>
+<wire x1="45.72" y1="83.82" x2="45.72" y2="93.98" width="0.1524" layer="91"/>
+<wire x1="45.72" y1="93.98" x2="27.94" y2="93.98" width="0.1524" layer="91"/>
+<pinref part="R3" gate="G$1" pin="2"/>
+</segment>
+</net>
