File: pcb_designs/arduino/gesture_control_robot_tx/gesture_control_robot_tx.sch (EAGLE design)
At the start: 29 parts, among them IC1 ATMEGA328, IC2 7805, IC3 HT12E, J2 transmitter, Q1 16MHZ

Commit message: modify
Parts:
- removed IC3: HT12E, microchip:PIC16F1826/27P
- removed J2: transmitter, con-amp:MTA04-100
- removed JP7, JP8: (no value), jumper:JP2E
- removed R3, R5, R6, R7: 1k, eagle-ltspice:R0204/7
- removed R8: 1ME, eagle-ltspice:R0204/7
- added TX: (no value), con-amp-quick:M04
Connections:
- removed net N$30: IC1.OBJ, IC3.RB4, R3.1
- removed net N$33: IC1.DA0/ECK, IC3.RB5, R5.1
- removed net N$34: IC1.BG, IC3.RB6, R7.2
- removed net N$35: IC1.STAT, IC3.RB7, R6.2
- removed net N$36: IC3.RA7, R8.1
- removed net N$37: IC3.RA6, R8.2
- removed net N$38: IC3.RA0, J2.3
- new net N$13: IC1.OUT, TX.2
- net N$4: now also TX.4; no longer IC3.RA1, J2.1, JP7.1, JP7.2, JP7.3, R3.2, R5.2, R6.1, R7.1
- net N$5: now also TX.3; no longer IC3.RA2, IC3.RA3, IC3.RA4, IC3.RA5/!MCLR!/VPP, IC3.RB0, IC3.RB1, IC3.RB2, IC3.RB3, IC3.VDD, IC3.VSS, J2.2, JP8.1, JP8.2, JP8.3
