File: pcb_designs/arduino/arduino_uno_pcb/uno.sch (EAGLE design)
At the start: 25 parts, among them IC1 ATMEGA328, IC2 7805, Q1 16MHZ

Commit message: modify
Parts:
- added JP9: (no value), jumper:JP2E
Connections:
- net N$7: now also JP9.1, JP9.2, JP9.3
Changed lines of the file:
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@@
 <?xml version="1.0" encoding="utf-8"?>
 <!DOCTYPE eagle SYSTEM "eagle.dtd">
-<eagle version="6.1">
+<eagle version="7.1.0">
 <drawing>
 <settings>
@@
 <part name="JP7" library="jumper" deviceset="JP2E" device=""/>
 <part name="JP8" library="jumper" deviceset="JP2E" device=""/>
+<part name="JP9" library="jumper" deviceset="JP2E" device=""/>
 </parts>
 <sheets>
@@
 <instance part="JP7" gate="1" x="83.82" y="76.2" rot="R270"/>
 <instance part="JP8" gate="1" x="33.02" y="17.78"/>
+<instance part="JP9" gate="1" x="33.02" y="83.82" rot="R180"/>
 </instances>
 <busses>
@@
 <pinref part="IC2" gate="A1" pin="VI"/>
 <junction x="35.56" y="86.36"/>
-<wire x1="35.56" y1="86.36" x2="27.94" y2="86.36" width="0.1524" layer="91"/>
+<wire x1="35.56" y1="86.36" x2="33.02" y2="86.36" width="0.1524" layer="91"/>
 <pinref part="C3" gate="G$1" pin="1"/>
+<wire x1="33.02" y1="86.36" x2="30.48" y2="86.36" width="0.1524" layer="91"/>
+<wire x1="30.48" y1="86.36" x2="27.94" y2="86.36" width="0.1524" layer="91"/>
 <wire x1="27.94" y1="86.36" x2="20.32" y2="86.36" width="0.1524" layer="91"/>
 <wire x1="20.32" y1="86.36" x2="20.32" y2="73.66" width="0.1524" layer="91"/>
@@
 <junction x="27.94" y="73.66"/>
 <pinref part="D1" gate="1" pin="C"/>
-</segment>
-</net>
+<pinref part="JP9" gate="1" pin="1"/>
+<pinref part="JP9" gate="1" pin="2"/>
+<junction x="33.02" y="86.36"/>
+<pinref part="JP9" gate="1" pin="3"/>
+<junction x="30.48" y="86.36"/>
+</segment>
+</net>
