File: pcb_designs/mini_projects/object_counter_0_to_99/object counter.brd (EAGLE design)
At the start: 75.9 x 77.5 mm, 13 parts, among them IC1 4033, IC2 4033

Commit message: add
Parts:
- added C1: (no value), capacitor-wima:C2.5-3
Connections:
- net N$1: now also C1.1
- net N$4: now also C1.2
Routing:
- net N$23: track 125.5 -> 130.6 mm
- net N$1: track 266.4 -> 270.2 mm
- net N$13: track 290.5 -> 287.3 mm
- net N$4: track 58.4 -> 61.0 mm
Other:
- board size 75.9 x 77.5 mm -> 87.3 x 77.5 mm
