File: pcb_designs/modules/adc_module/adc module.sch (EAGLE design)
At the start: 0 parts

Commit message: 
Parts:
- added C1: 150pf, capacitor-wima:C2,5-3
- added IC1: adc804, atmel:ATF16V8BP3
- added R1: 10k, eagle-ltspice:R0204/7
- added SL1: (no value), con-amp-quick:M12
- added SL2: (no value), con-amp-quick:M02
- added SL3: LM35, con-amp-quick:M03
- added SL4: (no value), con-amp-quick:M03
- added VR: 10k, resistor:R-TRIMM64P
Connections:
- new net N$1: IC1.O2, SL1.1
- new net N$10: C1.1, IC1.I3, R1.1
- new net N$12: IC1.I1, SL4.3
- new net N$13: IC1.I2, SL4.2
- new net N$14: IC1.I5, SL3.2
- new net N$15: IC1.I4, SL4.1
- new net N$17: IC1.I8, VR.S
- new net N$18: C1.2, IC1.CLK, IC1.GND, IC1.I6, IC1.I7, SL1.10, SL1.9, SL2.2, SL3.3, VR.A
- new net N$19: IC1.VCC, SL1.11, SL2.1, SL3.1, VR.E
- new net N$2: IC1.O3, SL1.2
- new net N$3: IC1.O4, SL1.3
- new net N$4: IC1.O5, SL1.4
- new net N$5: IC1.O6, SL1.5
- new net N$6: IC1.O7, SL1.6
- new net N$7: IC1.O8, SL1.7
- new net N$8: IC1.OE, SL1.8
- new net N$9: IC1.O1, R1.2
