File: micro_controllers/8051/projects/ultrasonic_distance_meter/pcb/ultrasonic_distance_meter.brd (EAGLE design)
At the start: 6.9 x 7 mm, 25 parts, among them IC1 AT89S51, IC2 7805TV

Commit message: 
Parts:
- CONNECTOR-1: value 4 pin -> ultrasonic sensor
Changed lines of the file:
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@@
 <layer number="21" name="tPlace" color="7" fill="1" visible="yes" active="yes"/>
 <layer number="22" name="bPlace" color="7" fill="1" visible="yes" active="yes"/>
-<layer number="23" name="tOrigins" color="15" fill="1" visible="no" active="yes"/>
+<layer number="23" name="tOrigins" color="15" fill="1" visible="yes" active="yes"/>
 <layer number="24" name="bOrigins" color="15" fill="1" visible="yes" active="yes"/>
 <layer number="25" name="tNames" color="7" fill="1" visible="yes" active="yes"/>
@@
 </element>
 <element name="C6" library="capacitor-wima" package="C2.5-6" value="0.1uf" x="24.13" y="8.89" rot="R270"/>
-<element name="CONNECTOR-1" library="con-amp-quick" package="04P" value="4 pin" x="63.5" y="13.97">
+<element name="CONNECTOR-1" library="con-amp-quick" package="04P" value="ultrasonic sensor" x="63.5" y="13.97">
 <attribute name="OC_NEWARK" value="unknown" x="63.5" y="13.97" size="1.778" layer="27" display="off"/>
 <attribute name="MPN" value="" x="63.5" y="13.97" size="1.778" layer="27" display="off"/>
