File: pcb_designs/mini_projects/demeler/demeler_pcb_new/demeler_pcb.brd (EAGLE design)
At the start: 246 x 152 mm, 36 parts, among them IC1 ATMEGA328, IC2 L293D, J2 1445055-5, Q1 16MHZ, X1 RJ45-6X, X2 KUSBVX

Commit message: 
Parts:
- removed SW1: (no value), special:EDG-02
- added ADAPTERPOER: (no value), jumper:JP1
- moved X2 70.0 mm to (111.7, 123.2)
- moved J2 60.0 mm to (88.6, 121.4)
- moved USB2LANOP 32.8 mm to (157.8, 125.0)
- moved JP3 32.8 mm to (189.8, 123.8)
- moved JP4 32.8 mm to (192.5, 127.0)
- moved JP7 26.7 mm to (116.4, 159.8)
- moved JP10 24.3 mm to (98.3, 160.2)
- moved JP8 20.9 mm to (78.4, 159.8)
- moved S1 14.4 mm to (102.8, 152.4)
- moved LED2 10.0 mm to (118.8, 154.2)
- moved R2 8.94 mm to (131.9, 154.6)
- moved JP9 6.58 mm to (146.8, 157.1), turned to 0 degrees
- moved R1 5.94 mm to (159.4, 153.6), turned to 90 degrees
- moved X1 4.47 mm to (214.4, 120.9)
- moved IC2 4.18 mm to (232.1, 145.9), turned to 180 degrees
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Connections:
- new net N$16: IC1.2, USB2SERIAL.2
- new net N$19: J2.5
- new net N$21: JP9.2, TX.4
- net +5V: no longer J2.1, X2.4
- net GND: no longer IC1.18, J1.1, J2.5, JP9.2, SW1.1, TX.4, X2.1
- net N$17: now also TX.1
- net N$20: no longer IC1.2, USB2SERIAL.2
- net N$23: no longer SW1.2
- net N$26: now also IC1.18
- net N$3: now also IC1.3, USB2SERIAL.1; no longer J1.3
- net N$4: no longer IC1.3, USB2SERIAL.1
Routing:
- net +5V: track 0.00 -> 357.2 mm
- net GND: track 0.00 -> 245.3 mm
- net N$26: track 0.00 -> 108.0 mm
- net N$25: track 0.00 -> 105.7 mm, vias 0 -> 2
- net N$24: track 0.00 -> 105.4 mm
- net N$13: track 0.00 -> 98.5 mm
- net N$16: track 0.00 -> 83.6 mm
- net N$15: track 0.00 -> 74.3 mm, vias 0 -> 2
- net N$3: track 0.00 -> 71.5 mm
- net N$12: track 0.00 -> 68.3 mm
- net N$14: track 0.00 -> 63.2 mm
- net N$8: track 0.00 -> 59.0 mm
- net N$10: track 0.00 -> 45.7 mm
- net N$11: track 0.00 -> 44.6 mm
- net N$18: track 0.00 -> 33.1 mm
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- added copper zone on layer 16, net N$22
